File: SERV.brd (EAGLE design)
At the start: 57 x 57 mm, 69 parts

Commit message: Исправлено
Parts:
- added C20: 0.1uF, Discrete:0603
- added R2: 10K, Discrete:0603
- added R27: 10K*, Discrete:0603
- D1: value (none) -> BZV55-C3V9
- R15: value 10K -> 10K*
- moved R15 0.63 mm to (55.9, 36.0)
Connections:
- new net N$2: R2.2, STM32.44
- new net N$3: C20.2, MPU.10
- new net N$4: MPU.22, R27.1
- net 3.3V: now also R27.2; no longer MPU.22
- net GND: now also C20.1, R2.1; no longer STM32.44
Routing:
- net N$2: track 0.00 -> 12.9 mm, vias 0 -> 2
- net N$4: track 0.00 -> 6.14 mm, vias 0 -> 1
- net GND: track 136.2 -> 130.7 mm, vias 45 -> 46
- net N$3: track 0.00 -> 3.18 mm
Other:
- board text added: "Curator - Krestovnikov Designer - Luzhetsky Board version - 0.2"
- board text added: "SERV"
- board text removed: "SERV.BTN.LUZHETSKII.0.1"

Commit message: fixed
Parts:
- C11, C12, C13, C14, C15, C16, C17, C18, C19, C2, C20, C3, C4, C5, C6, C7, C9, R1, R10, R11, R12, R13, R14, R15, R18, R19, R2, R20, R21, R22, R23, R24, R25, R26, R27, R3, R4, R5, R6, R7, R8, R9: device Discrete:0603 -> discrete:0603
- R16, R17: value 10K -> 4.7k; device Discrete:0603 -> discrete:0603
- moved U$1 2.16 mm to (23.6, 25.8), turned to 333.6 degrees
Connections:
- net GND: now also MPU.25
Routing:
- net GND: track 130.7 -> 379.5 mm
- net 3.3V: track 92.8 -> 147.5 mm, vias 13 -> 14
- net PHASE_B: track 0.00 -> 27.2 mm, vias 0 -> 6
- net PHASE_A: track 0.00 -> 23.5 mm, vias 0 -> 6
- net PHASE_B1: track 22.4 -> 0.00 mm, vias 6 -> 0
- net PHASE_A1: track 20.2 -> 0.00 mm, vias 6 -> 0
- net PHASE_C: track 0.00 -> 17.3 mm, vias 0 -> 6
- net PHASE_C1: track 15.8 -> 0.00 mm, vias 6 -> 0
- net VIN: track 82.4 -> 97.0 mm
- net N$51: track 12.7 -> 11.4 mm
- net SDA: track 41.8 -> 40.9 mm
- net ACTIVATE_A: track 40.1 -> 39.3 mm
- net 3.3V_S: track 20.5 -> 19.9 mm
- net N$31: track 6.72 -> 6.20 mm
- removed copper zone on layer 2, net 3.3V
- removed copper zone on layer 1, net VIN
